Commit message: Fix 6 simulation issues: wheel axis, sinking, control direction, bridge types, slam scan topic, and xacro quoting
- Fix xacro parsing: quoted collision_rpy default values in wheel_type1/2.xacro
- Fix wheel rotation axis: changed from Z-axis (0 0 1) to Y-axis (0 -1 0)
- Fix wheel sinking: corrected base_footprint z-offset with wheel_vertical_offset, added collision_rpy to rotate cylinder horizontal
- Fix keyboard control: unified axis="0 -1 0" with swapped DiffDrive left/right joints
- Fix slam scan topic: changed /scan to /front/scan in slam_toolbox_params.yaml
- Fix bridge message types: unified ignition.msgs to gz.msgs for odom/tf/joint_states
- Add tf_static_relay.py to forward /tf_static to /tf (attempts to fix SLAM ghosting)
- Add transform_timeout and transform_tolerance to SLAM config

Unresolved: SLAM pose not updating (ghosting) — see .github/ISSUES/slam-ghosting.md

File: src/scout_mini_dual_lidar_gazebo/urdf/scout_mini_gazebo.xacro (robot description, xacro)
@@ -21,5 +21,5 @@
     <link name="base_link">
         <visual>
-            <origin xyz="0 0 0" rpy="0 0 0" />
+            <origin xyz="0 0 0" rpy="0 0 3.14159" />
             <geometry>
                 <mesh filename="${mesh_prefix}/meshes/base_link.dae" />
@@ -41,5 +41,5 @@
     <link name="base_footprint"/>
     <joint name="base_footprint_joint" type="fixed">
-        <origin xyz="0 0 ${-wheel_radius}" rpy="0 0 0" />
+        <origin xyz="0 0 ${wheel_vertical_offset - wheel_radius}" rpy="0 0 0" />
         <parent link="base_link" />
         <child link="base_footprint" />
@@ -49,5 +49,5 @@
             <mass value="25" />
             <origin xyz="0.0 0.0 0.0" />
-            <inertia ixx="1.0" ixy="0" ixz="0" iyy="2.0" iyz="0" izz="1.5" />
+            <inertia ixx="0.323" ixy="0" ixz="0" iyy="0.948" iyz="0" izz="1.135" />
         </inertial>
     </link>
@@ -57,16 +57,18 @@
         <child link="inertial_link" />
     </joint>
-    <!-- Scout Mini wheel macros -->
-    <xacro:scout_wheel_type1 wheel_prefix="front_right">
-        <origin xyz="${wheelbase/2} ${-track/2} ${wheel_vertical_offset}" rpy="3.14 0 0" />
+    <!-- 4-wheel direct drive (no mimic) -->
+    <!-- All wheels share same axis "0 -1 0" (Y-axis). -->
+    <!-- collision_rpy rotates cylinder from vertical to horizontal to match wheel shape. -->
+    <xacro:scout_wheel_type1 wheel_prefix="front_left" axis_xyz="0 -1 0" collision_rpy="1.5708 0 0">
+        <origin xyz="${wheelbase/2} ${track/2} ${wheel_vertical_offset}" rpy="0 0 0"/>
     </xacro:scout_wheel_type1>
-    <xacro:scout_wheel_type2 wheel_prefix="front_left">
-        <origin xyz="${wheelbase/2} ${track/2} ${wheel_vertical_offset}" rpy="0 0 0" />
+    <xacro:scout_wheel_type2 wheel_prefix="front_right" axis_xyz="0 -1 0" collision_rpy="1.5708 0 0">
+        <origin xyz="${wheelbase/2} ${-track/2} ${wheel_vertical_offset}" rpy="0 0 0"/>
     </xacro:scout_wheel_type2>
-    <xacro:scout_wheel_type1 wheel_prefix="rear_left">
-        <origin xyz="${-wheelbase/2} ${track/2} ${wheel_vertical_offset}" rpy="0 0 0" />
+    <xacro:scout_wheel_type1 wheel_prefix="rear_left" axis_xyz="0 -1 0" collision_rpy="1.5708 0 0">
+        <origin xyz="${-wheelbase/2} ${track/2} ${wheel_vertical_offset}" rpy="0 0 0"/>
     </xacro:scout_wheel_type1>
-    <xacro:scout_wheel_type2 wheel_prefix="rear_right">
-        <origin xyz="${-wheelbase/2} ${-track/2} ${wheel_vertical_offset}" rpy="3.14 0 0" />
+    <xacro:scout_wheel_type2 wheel_prefix="rear_right" axis_xyz="0 -1 0" collision_rpy="1.5708 0 0">
+        <origin xyz="${-wheelbase/2} ${-track/2} ${wheel_vertical_offset}" rpy="0 0 0"/>
     </xacro:scout_wheel_type2>
     <!-- Front LiDAR (RS-AIRY) -->
@@ -129,8 +131,12 @@
     <gazebo>
         <plugin filename="gz-sim-diff-drive-system" name="gz::sim::systems::DiffDrive">
-            <left_joint>rear_left_wheel</left_joint>
-            <right_joint>rear_right_wheel</right_joint>
+            <left_joint>front_right_wheel</left_joint>
+            <left_joint>rear_right_wheel</left_joint>
+            <right_joint>front_left_wheel</right_joint>
+            <right_joint>rear_left_wheel</right_joint>
             <wheel_separation>${track}</wheel_separation>
             <wheel_radius>${wheel_radius}</wheel_radius>
+            <max_wheel_torque>20</max_wheel_torque>
+            <max_linear_acceleration>1.0</max_linear_acceleration>
             <topic>/cmd_vel</topic>
             <odom_topic>/odom</odom_topic>
@@ -138,7 +144,7 @@
             <odom_publish_frequency>50</odom_publish_frequency>
             <odom_frame>odom</odom_frame>
-            <robot_base_frame>base_footprint</robot_base_frame>
-            <linear_velocity_limit>2.0</linear_velocity_limit>
-            <angular_velocity_limit>3.0</angular_velocity_limit>
+            <robot_base_frame>base_link</robot_base_frame>
+            <max_linear_velocity>2.0</max_linear_velocity>
+            <max_angular_velocity>3.0</max_angular_velocity>
         </plugin>
     </gazebo>

Commit message: fix: switch to scout_mini.urdf, correct wheel axes, add IMU odometry correction
- Switch from scout_mini.xacro to scout_mini.urdf with matching properties
- Fix wheel axis directions (unified -Y in base_link frame)
- Swap DiffDrive left/right joints + use +track for correct odometry
- Simplify collision bodies: base_link mesh→box, wheels mesh→cylinder
- Reduce mu2 (lateral friction) to 0.5 for skid-steer simulation
- Add IMU-corrected odometry (imu_odom_corrector.py) to fix rotation drift
- Add auto_path_driver.py for automated test path execution
- Tune SLAM: enable loop closure, increase keyframe thresholds, occ_thresh→0.35
- Lower LiDAR positions to match Scout Mini chassis height
- Fix wheel_radius in scout_diff_drive_controller.py (0.101→0.08)
- Optimize physics: max_step_size 0.005, quick solver, RTF stabilization

File: src/scout_mini_dual_lidar_gazebo/urdf/scout_mini_gazebo.xacro (robot description, xacro)
@@ -2,41 +2,30 @@
 <robot name="scout_mini"
     xmlns:xacro="http://ros.org/wiki/xacro">
-    <xacro:arg name="robot_namespace" default="/" />
-    <xacro:arg name="mesh_prefix" default="package://scout_description" />
-    <xacro:include filename="$(find scout_description)/urdf/scout_wheel_type1.xacro" />
-    <xacro:include filename="$(find scout_description)/urdf/scout_wheel_type2.xacro" />
-    <!-- Variables for Scout Mini -->
-    <xacro:property name="M_PI" value="3.14159"/>
-    <xacro:property name="mesh_prefix" value="$(arg mesh_prefix)" />
-    <!-- Vehicle Geometries - Scout Mini dimensions -->
-    <xacro:property name="base_x_size" value="0.650" />
-    <xacro:property name="base_y_size" value="0.350" />
-    <xacro:property name="base_z_size" value="0.180" />
-    <xacro:property name="wheelbase" value="0.380" />
-    <xacro:property name="track" value="0.520" />
-    <xacro:property name="wheel_vertical_offset" value="-0.060" />
-    <xacro:property name="wheel_length" value="0.100" />
-    <xacro:property name="wheel_radius" value="0.145" />
-    <!-- Base link -->
-    <link name="base_link">
-        <visual>
-            <origin xyz="0 0 0" rpy="0 0 3.14159" />
-            <geometry>
-                <mesh filename="${mesh_prefix}/meshes/base_link.dae" />
-            </geometry>
-        </visual>
-        <collision>
-            <origin xyz="0 0 0.008" rpy="0 0 0" />
-            <geometry>
-                <box size="${base_x_size} ${base_y_size} ${base_z_size}"/>
-            </geometry>
-        </collision>
-        <collision>
-            <origin xyz="0 0 ${base_z_size/6}" rpy="0 0 0" />
-            <geometry>
-                <box size="${base_x_size/6} ${base_y_size*1.65} ${base_z_size/3}"/>
-            </geometry>
-        </collision>
-    </link>
+    <!-- ============================================================ -->
+    <!-- Include base chassis + wheels from URDF                       -->
+    <!-- scout_mini.urdf was generated from mini.xacro with values:    -->
+    <!--   wheelbase=0.463951  track=0.416503                         -->
+    <!--   wheel_vertical_offset=-0.100998  wheel_radius=0.08         -->
+    <!--   base 0.62 x 0.585 x 0.235                                 -->
+    <!-- ============================================================ -->
+    <xacro:include filename="$(find scout_description)/urdf/scout_mini.urdf" />
+    <!-- ============================================================ -->
+    <!-- Properties matching URDF values (for downstream use)          -->
+    <!-- ============================================================ -->
+    <xacro:property name="base_x_size" value="0.62" />
+    <xacro:property name="base_y_size" value="0.585" />
+    <xacro:property name="base_z_size" value="0.235" />
+    <xacro:property name="wheelbase" value="0.463951" />
+    <xacro:property name="track" value="0.416503" />
+    <xacro:property name="wheel_vertical_offset" value="-0.100998" />
+    <xacro:property name="wheel_radius" value="0.08" />
+    <xacro:property name="wheel_diameter" value="0.16" />
+    <!-- ============================================================ -->
+    <!-- Gazebo configuration (not in URDF)                            -->
+    <!-- ============================================================ -->
+    <xacro:include filename="$(find scout_description)/urdf/scout_mini.gazebo" />
+    <!-- ============================================================ -->
+    <!-- base_footprint (not in URDF)                                  -->
+    <!-- ============================================================ -->
     <link name="base_footprint"/>
     <joint name="base_footprint_joint" type="fixed">
@@ -45,32 +34,7 @@
         <child link="base_footprint" />
     </joint>
-    <link name="inertial_link">
-        <inertial>
-            <mass value="25" />
-            <origin xyz="0.0 0.0 0.0" />
-            <inertia ixx="0.323" ixy="0" ixz="0" iyy="0.948" iyz="0" izz="1.135" />
-        </inertial>
-    </link>
-    <joint name="inertial_joint" type="fixed">
-        <origin xyz="0 0 0" rpy="0 0 0" />
-        <parent link="base_link" />
-        <child link="inertial_link" />
-    </joint>
-    <!-- 4-wheel direct drive (no mimic) -->
-    <!-- All wheels share same axis "0 -1 0" (Y-axis). -->
-    <!-- collision_rpy rotates cylinder from vertical to horizontal to match wheel shape. -->
-    <xacro:scout_wheel_type1 wheel_prefix="front_left" axis_xyz="0 -1 0" collision_rpy="1.5708 0 0">
-        <origin xyz="${wheelbase/2} ${track/2} ${wheel_vertical_offset}" rpy="0 0 0"/>
-    </xacro:scout_wheel_type1>
-    <xacro:scout_wheel_type2 wheel_prefix="front_right" axis_xyz="0 -1 0" collision_rpy="1.5708 0 0">
-        <origin xyz="${wheelbase/2} ${-track/2} ${wheel_vertical_offset}" rpy="0 0 0"/>
-    </xacro:scout_wheel_type2>
-    <xacro:scout_wheel_type1 wheel_prefix="rear_left" axis_xyz="0 -1 0" collision_rpy="1.5708 0 0">
-        <origin xyz="${-wheelbase/2} ${track/2} ${wheel_vertical_offset}" rpy="0 0 0"/>
-    </xacro:scout_wheel_type1>
-    <xacro:scout_wheel_type2 wheel_prefix="rear_right" axis_xyz="0 -1 0" collision_rpy="1.5708 0 0">
-        <origin xyz="${-wheelbase/2} ${-track/2} ${wheel_vertical_offset}" rpy="0 0 0"/>
-    </xacro:scout_wheel_type2>
-    <!-- Front LiDAR (RS-AIRY) -->
+    <!-- ============================================================ -->
+    <!-- Front LiDAR (RS-AIRY)                                        -->
+    <!-- ============================================================ -->
     <link name="front_lidar_link">
         <visual>
@@ -96,9 +60,11 @@
     </link>
     <joint name="front_lidar_joint" type="fixed">
-        <origin xyz="${base_x_size/2 - 0.08} 0.0 ${base_z_size/2 + 0.05}" rpy="0 0 0" />
+        <origin xyz="${base_x_size/2 - 0.08} 0.0 ${base_z_size/2 - 0.03}" rpy="0 0 0" />
         <parent link="base_link" />
         <child link="front_lidar_link" />
     </joint>
-    <!-- Rear LiDAR (RS-AIRY) -->
+    <!-- ============================================================ -->
+    <!-- Rear LiDAR (RS-AIRY)                                         -->
+    <!-- ============================================================ -->
     <link name="rear_lidar_link">
         <visual>
@@ -124,94 +90,7 @@
     </link>
     <joint name="rear_lidar_joint" type="fixed">
-        <origin xyz="${-base_x_size/2 + 0.08} 0.0 ${base_z_size/2 + 0.05}" rpy="0 0 3.14159" />
+        <origin xyz="${-base_x_size/2 + 0.08} 0.0 ${base_z_size/2 - 0.03}" rpy="0 0 3.14159" />
         <parent link="base_link" />
         <child link="rear_lidar_link" />
     </joint>
-    <!-- Gazebo differential drive plugin -->
-    <gazebo>
-        <plugin filename="gz-sim-diff-drive-system" name="gz::sim::systems::DiffDrive">
-            <left_joint>front_right_wheel</left_joint>
-            <left_joint>rear_right_wheel</left_joint>
-            <right_joint>front_left_wheel</right_joint>
-            <right_joint>rear_left_wheel</right_joint>
-            <wheel_separation>${track}</wheel_separation>
-            <wheel_radius>${wheel_radius}</wheel_radius>
-            <max_wheel_torque>20</max_wheel_torque>
-            <max_linear_acceleration>1.0</max_linear_acceleration>
-            <topic>/cmd_vel</topic>
-            <odom_topic>/odom</odom_topic>
-            <tf_topic>/tf</tf_topic>
-            <odom_publish_frequency>50</odom_publish_frequency>
-            <odom_frame>odom</odom_frame>
-            <robot_base_frame>base_link</robot_base_frame>
-            <max_linear_velocity>2.0</max_linear_velocity>
-            <max_angular_velocity>3.0</max_angular_velocity>
-        </plugin>
-    </gazebo>
-    <!-- Gazebo joint state publisher -->
-    <gazebo>
-        <plugin filename="gz-sim-joint-state-publisher-system" name="gz::sim::systems::JointStatePublisher">
-            <topic>/joint_states</topic>
-        </plugin>
-    </gazebo>
-    <!-- Front LiDAR Gazebo sensor plugin -->
-    <gazebo reference="front_lidar_link">
-        <sensor name="front_lidar_sensor" type="gpu_ray">
-            <pose>0 0 0 0 0 0</pose>
-            <visualize>true</visualize>
-            <update_rate>5</update_rate>
-            <always_on>true</always_on>
-            <ray>
-                <scan>
-                    <horizontal>
-                        <samples>360</samples>
-                        <resolution>1.0</resolution>
-                        <min_angle>-3.14159</min_angle>
-                        <max_angle>3.14159</max_angle>
-                    </horizontal>
-                </scan>
-                <range>
-                    <min>0.1</min>
-                    <max>25.0</max>
-                    <resolution>0.01</resolution>
-                </range>
-                <noise>
-                    <type>gaussian</type>
-                    <mean>0.0</mean>
-                    <stddev>0.01</stddev>
-                </noise>
-            </ray>
-            <topic>/front/scan</topic>
-        </sensor>
-    </gazebo>
-    <!-- Rear LiDAR Gazebo sensor plugin -->
-    <gazebo reference="rear_lidar_link">
-        <sensor name="rear_lidar_sensor" type="gpu_ray">
-            <pose>0 0 0 0 0 0</pose>
-            <visualize>true</visualize>
-            <update_rate>5</update_rate>
-            <always_on>true</always_on>
-            <ray>
-                <scan>
-                    <horizontal>
-                        <samples>360</samples>
-                        <resolution>1.0</resolution>
-                        <min_angle>-3.14159</min_angle>
-                        <max_angle>3.14159</max_angle>
-                    </horizontal>
-                </scan>
-                <range>
-                    <min>0.1</min>
-                    <max>25.0</max>
-                    <resolution>0.01</resolution>
-                </range>
-                <noise>
-                    <type>gaussian</type>
-                    <mean>0.0</mean>
-                    <stddev>0.01</stddev>
-                </noise>
-            </ray>
-            <topic>/rear/scan</topic>
-        </sensor>
-    </gazebo>
 </robot>
