Commit message: feat: complete stage-5 IoT pick-and-place pipeline with EKF odometry
- Add EKF fusion (robot_localization) merging wheel odometry with IMU
  yaw to eliminate cornering drift
- Add ManipulationNode: Piper arm waypoint execution, gripper control,
  DetachableJoint attach/detach for Gazebo Sim
- Add iot_device.sdf and pickup_table.sdf world models
- Add proximity-stop logic in DeploymentApproachNode: treat navigation
  abort near target as arrival (robot bumped into table/obstacle)
- Tune laser self-filter hull to cover Piper arm envelope, preventing
  false inflation layer obstacles
- Tune pick/place arm poses: device spawns on chassis top between arm
  base and front LiDAR, place pose extends past front bumper
- Fix Gazebo launch: add -r flag to unpause simulation
- Add AMCL automatic initial pose setup
- Fix cmd_vel type: use Twist (not TwistStamped) for DiffDrive
- Simplify imu_odom_corrector to frame_id cleanup only, EKF handles
  the sensor fusion

File: src/piper_description/urdf/piper_description.xacro (robot description, xacro)
@@ -503,7 +503,140 @@
       effort="10"
       velocity="1" />
-  </joint>
-  <!-- ros2_control transmissions and gazebo_ros2_control plugin intentionally omitted:
-       stage 1 uses joint_state_publisher only; control stack added in stage 5 -->
+    <!-- Passive finger: follows joint7 in opposition (axis 0 0 -1) -->
+    <mimic joint="joint7" multiplier="1" offset="0" />
+  </joint>
+  <!-- ============================================================ -->
+  <!-- Stage 5: ros2_control transmissions                          -->
+  <!-- SimpleTransmission + PositionJointInterface for joint1..6    -->
+  <!-- and gripper joint7 (joint8 is a passive mimic finger).       -->
+  <!-- Existing <dynamics damping friction> settings are kept.      -->
+  <!-- ============================================================ -->
+  <transmission name="tran_joint1">
+    <type>transmission_interface/SimpleTransmission</type>
+    <joint name="joint1">
+      <hardwareInterface>hardware_interface/PositionJointInterface</hardwareInterface>
+    </joint>
+    <actuator name="motor_joint1">
+      <hardwareInterface>hardware_interface/PositionJointInterface</hardwareInterface>
+      <mechanicalReduction>1</mechanicalReduction>
+    </actuator>
+  </transmission>
+  <transmission name="tran_joint2">
+    <type>transmission_interface/SimpleTransmission</type>
+    <joint name="joint2">
+      <hardwareInterface>hardware_interface/PositionJointInterface</hardwareInterface>
+    </joint>
+    <actuator name="motor_joint2">
+      <hardwareInterface>hardware_interface/PositionJointInterface</hardwareInterface>
+      <mechanicalReduction>1</mechanicalReduction>
+    </actuator>
+  </transmission>
+  <transmission name="tran_joint3">
+    <type>transmission_interface/SimpleTransmission</type>
+    <joint name="joint3">
+      <hardwareInterface>hardware_interface/PositionJointInterface</hardwareInterface>
+    </joint>
+    <actuator name="motor_joint3">
+      <hardwareInterface>hardware_interface/PositionJointInterface</hardwareInterface>
+      <mechanicalReduction>1</mechanicalReduction>
+    </actuator>
+  </transmission>
+  <transmission name="tran_joint4">
+    <type>transmission_interface/SimpleTransmission</type>
+    <joint name="joint4">
+      <hardwareInterface>hardware_interface/PositionJointInterface</hardwareInterface>
+    </joint>
+    <actuator name="motor_joint4">
+      <hardwareInterface>hardware_interface/PositionJointInterface</hardwareInterface>
+      <mechanicalReduction>1</mechanicalReduction>
+    </actuator>
+  </transmission>
+  <transmission name="tran_joint5">
+    <type>transmission_interface/SimpleTransmission</type>
+    <joint name="joint5">
+      <hardwareInterface>hardware_interface/PositionJointInterface</hardwareInterface>
+    </joint>
+    <actuator name="motor_joint5">
+      <hardwareInterface>hardware_interface/PositionJointInterface</hardwareInterface>
+      <mechanicalReduction>1</mechanicalReduction>
+    </actuator>
+  </transmission>
+  <transmission name="tran_joint6">
+    <type>transmission_interface/SimpleTransmission</type>
+    <joint name="joint6">
+      <hardwareInterface>hardware_interface/PositionJointInterface</hardwareInterface>
+    </joint>
+    <actuator name="motor_joint6">
+      <hardwareInterface>hardware_interface/PositionJointInterface</hardwareInterface>
+      <mechanicalReduction>1</mechanicalReduction>
+    </actuator>
+  </transmission>
+  <transmission name="tran_joint7">
+    <type>transmission_interface/SimpleTransmission</type>
+    <joint name="joint7">
+      <hardwareInterface>hardware_interface/PositionJointInterface</hardwareInterface>
+    </joint>
+    <actuator name="motor_joint7">
+      <hardwareInterface>hardware_interface/PositionJointInterface</hardwareInterface>
+      <mechanicalReduction>1</mechanicalReduction>
+    </actuator>
+  </transmission>
+  <!-- joint8 is the passive finger: mimic joint7 so it closes in -->
+  <!-- opposition without its own controller (kept out of           -->
+  <!-- ros2_control / transmissions).                               -->
+  <xacro:property name="_stage5_mimic" value="true" />
+  <!-- ============================================================ -->
+  <!-- Stage 5: ros2_control system, driven by ign_ros2_control     -->
+  <!-- (Gazebo Sim Fortress). controller_manager runs inside the    -->
+  <!-- simulator; controllers are loaded by spawners in the launch. -->
+  <!-- ============================================================ -->
+  <ros2_control name="PiperSimSystem" type="system">
+    <hardware>
+      <plugin>ign_ros2_control/IgnitionSystem</plugin>
+    </hardware>
+    <joint name="joint1">
+      <command_interface name="position"/>
+      <state_interface name="position"/>
+      <state_interface name="velocity"/>
+    </joint>
+    <joint name="joint2">
+      <command_interface name="position"/>
+      <state_interface name="position"/>
+      <state_interface name="velocity"/>
+    </joint>
+    <joint name="joint3">
+      <command_interface name="position"/>
+      <state_interface name="position"/>
+      <state_interface name="velocity"/>
+    </joint>
+    <joint name="joint4">
+      <command_interface name="position"/>
+      <state_interface name="position"/>
+      <state_interface name="velocity"/>
+    </joint>
+    <joint name="joint5">
+      <command_interface name="position"/>
+      <state_interface name="position"/>
+      <state_interface name="velocity"/>
+    </joint>
+    <joint name="joint6">
+      <command_interface name="position"/>
+      <state_interface name="position"/>
+      <state_interface name="velocity"/>
+    </joint>
+    <joint name="joint7">
+      <command_interface name="position"/>
+      <state_interface name="position"/>
+      <state_interface name="velocity"/>
+    </joint>
+  </ros2_control>
+  <!-- ign_ros2_control plugin: starts a controller_manager inside  -->
+  <!-- Gazebo Sim for this model. The parameters file supplies      -->
+  <!-- controller definitions (piper_controllers.yaml).             -->
+  <gazebo>
+    <plugin filename="ign_ros2_control-system" name="ign_ros2_control::IgnitionROS2ControlPlugin">
+      <parameters>$(find scout_mini_dual_lidar_gazebo)/config/piper_controllers.yaml</parameters>
+    </plugin>
+  </gazebo>
   <!-- <gazebo reference="base_link">
     <material>Gazebo/Black</material>

File: src/scout_mini_dual_lidar_gazebo/urdf/piper_mount.xacro (robot description, xacro)
@@ -16,3 +16,24 @@
         <child link="piper_base_link" />
     </joint>
+    <!-- ============================================================ -->
+    <!-- Stage 5: DetachableJoint system plugin on the parent model    -->
+    <!-- (scout_mini). It welds <child_link> of <child_model> to the    -->
+    <!-- gripper on an Empty message to <attach_topic>, and breaks the  -->
+    <!-- weld on a message to <detach_topic>, leaving the device where  -->
+    <!-- it was released. Triggered via gz-transport `ign topic` CLI.   -->
+    <!-- NOTE: gripper_base is a fixed joint so sdformat lumps it into   -->
+    <!-- link6 and it is NOT a real link in SDF; link7 (a gripper        -->
+    <!-- finger) is a genuine link at the gripper tip, so we weld to it. -->
+    <!-- ============================================================ -->
+    <gazebo>
+        <plugin filename="ignition-gazebo-detachable-joint-system"
+                name="gz::sim::systems::DetachableJoint">
+            <parent_link>link7</parent_link>
+            <child_model>iot_device</child_model>
+            <child_link>iot_device_link</child_link>
+            <attach_topic>/iot_device/attach</attach_topic>
+            <detach_topic>/iot_device/detach</detach_topic>
+            <output_topic>/iot_device/detachable_joint/state</output_topic>
+        </plugin>
+    </gazebo>
 </robot>

Commit message: feat: Stage 3-7 取货/放置/端到端集成完成
- 修复 joint2/3 无法运动（damping/friction 10.0→1.0）
- 取货流程新增开爪步骤（home→open→pick_above→pick→close→attach→carry）
- 放置流程实现 set_pose 瞬移设备到目标位姿
- 实现 mock_pick 模式跳过取货直接验证放置
- deployment_shelf 改为悬空桌面（0.40×0.30m，支柱后置避免卡住机器人）
- 候选半径调整为 0.25~0.50m，导航无障碍
- waypoints joint5 超限修复
- 添加校准/调试工具脚本
- 端到端全链路：取货→导航→放置→DEPLOYMENT_COMPLETE 验证通过

File: src/piper_description/urdf/piper_description.xacro (robot description, xacro)
@@ -83,5 +83,5 @@
       effort="100"
       velocity="5" />
-    <dynamics damping="10.0" friction="10.0" />
+    <dynamics damping="1.0" friction="1.0" />
   </joint>
   <link
@@ -134,5 +134,5 @@
       effort="100"
       velocity="5" />
-    <dynamics damping="10.0" friction="10.0" />
+    <dynamics damping="1.0" friction="1.0" />
   </joint>
   <link
@@ -185,5 +185,5 @@
       effort="100"
       velocity="5" />
-    <dynamics damping="10.0" friction="10.0" />
+    <dynamics damping="1.0" friction="1.0" />
   </joint>
   <link
@@ -235,5 +235,5 @@
       effort="100"
       velocity="5" />
-    <dynamics damping="10.0" friction="10.0" />
+    <dynamics damping="1.0" friction="1.0" />
   </joint>
   <link
@@ -285,5 +285,5 @@
       effort="100"
       velocity="5" />
-    <dynamics damping="10.0" friction="10.0" />
+    <dynamics damping="1.0" friction="1.0" />
   </joint>
   <link
@@ -335,5 +335,5 @@
       effort="100"
       velocity="3" />
-    <dynamics damping="10.0" friction="10.0" />
+    <dynamics damping="1.0" friction="1.0" />
   </joint>
   <link
